File: UV Exposure/UV Exposure.kicad_pcb (KiCad board)
At the start: 2 copper layers, 102 x 90 mm, 96 parts, among them P1 Conn_01x01, P2 Conn_01x01

Commit message: add logo and rearange track
Parts:
- added REF**: drawing, UV Exposure:drawing, B.Cu at (90.4, 88.9)
- added REF**: OSHW-Logo2_7.3x6mm_Copper, Symbol:OSHW-Logo2_7.3x6mm_Copper, B.Cu at (89.9, 54.9)
Other:
- board text removed: "UV Exposure Light"
